File: lifesense-pcb.sch (KiCad schematic (older format))
At the start: 2 parts

Commit message: Adding msp430 and cc3000 footprint.
Parts:
- added ??1: MSP430F5529, symbol MSP430F5529
- added IC1: CC3000, symbol CC3000
- gave numbers to parts that had none: 2
Changed lines of the file:
@@
 LIBS:contrib
 LIBS:valves
+LIBS:texasF5529
+LIBS:ti-ic
+LIBS:lifesense-pcb-cache
 EELAYER 24 0
 EELAYER END
@@
 $EndDescr
 $Comp
-L LED D?
+L LED D1
 U 1 1 5389F798
 P 4150 2050
-F 0 "D?" H 4150 2150 50  0000 C CNN
+F 0 "D1" H 4150 2150 50  0000 C CNN
 F 1 "LED" H 4150 1950 50  0000 C CNN
 F 2 "" H 4150 2050 60  0000 C CNN
@@
 $EndComp
 $Comp
-L R R?
+L R R1
 U 1 1 5389F825
 P 4150 2600
-F 0 "R?" V 4230 2600 40  0000 C CNN
+F 0 "R1" V 4230 2600 40  0000 C CNN
 F 1 "R" V 4157 2601 40  0000 C CNN
 F 2 "" V 4080 2600 30  0000 C CNN
@@
 	4150 2850 4150 3150
 $Comp
-L GND #PWR?
+L GND #PWR2
 U 1 1 5389F8DA
 P 4150 3150
-F 0 "#PWR?" H 4150 3150 30  0001 C CNN
+F 0 "#PWR2" H 4150 3150 30  0001 C CNN
 F 1 "GND" H 4150 3080 30  0001 C CNN
 F 2 "" H 4150 3150 60  0000 C CNN
@@
 $EndComp
 $Comp
-L VCC #PWR?
+L VCC #PWR1
 U 1 1 5389F944
 P 4150 1600
-F 0 "#PWR?" H 4150 1700 30  0001 C CNN
+F 0 "#PWR1" H 4150 1700 30  0001 C CNN
 F 1 "VCC" H 4150 1700 30  0000 C CNN
 F 2 "" H 4150 1600 60  0000 C CNN
@@
 Wire Wire Line
 	4150 2350 4150 2250
+$Comp
+L MSP430F5529 ??1
+U 1 1 5394CA66
+P 7400 3300
+F 0 "??1" H 7400 3300 60  0000 C CNN
+F 1 "MSP430F5529" H 7400 3300 60  0000 C CNN
+F 2 "" H 7400 3300 60  0000 C CNN
+F 3 "" H 7400 3300 60  0000 C CNN
+	1    7400 3300
+	1    0    0    -1
+$EndComp
+$Comp
+L CC3000 IC1
+U 1 1 5394D013
+P 3000 5500
+F 0 "IC1" H 2150 6950 60  0000 C CNN
+F 1 "CC3000" H 3750 6950 60  0000 C CNN
+F 2 "" H 2900 5400 60  0001 C CNN
+F 3 "http://www.ti.com/lit/gpn/cc3000" H 3000 3600 60  0001 C CNN
+F 4 "296-35512-1-ND" H 3000 3400 60  0001 C CNN "Distrib. Part"
+F 5 "CC3000MOD" H 3000 3700 60  0001 C CNN "Manuf. Part"
+F 6 "Digikey" H 3000 3500 60  0001 C CNN "Distributor"
+F 7 "TI" H 3000 3800 60  0001 C CNN "Manufacturer"
+	1    3000 5500
+	1    0    0    -1
+$EndComp
 $EndSCHEMATC

Commit message: moving to tiva-c TM4C123GH6PM chip
Parts:
- removed ??1: MSP430F5529, symbol MSP430F5529
- added U1: TM4C1230H6PM, LQFP64, symbol TM4C1230H6PM
Changed lines of the file:
@@
 	4150 2850 4150 3150
 $Comp
-L GND #PWR2
+L GND #PWR01
 U 1 1 5389F8DA
 P 4150 3150
-F 0 "#PWR2" H 4150 3150 30  0001 C CNN
+F 0 "#PWR01" H 4150 3150 30  0001 C CNN
 F 1 "GND" H 4150 3080 30  0001 C CNN
 F 2 "" H 4150 3150 60  0000 C CNN
@@
 $EndComp
 $Comp
-L VCC #PWR1
+L VCC #PWR02
 U 1 1 5389F944
 P 4150 1600
-F 0 "#PWR1" H 4150 1700 30  0001 C CNN
+F 0 "#PWR02" H 4150 1700 30  0001 C CNN
 F 1 "VCC" H 4150 1700 30  0000 C CNN
 F 2 "" H 4150 1600 60  0000 C CNN
@@
 Wire Wire Line
 	4150 2350 4150 2250
-$Comp
-L MSP430F5529 ??1
-U 1 1 5394CA66
-P 7400 3300
-F 0 "??1" H 7400 3300 60  0000 C CNN
-F 1 "MSP430F5529" H 7400 3300 60  0000 C CNN
-F 2 "" H 7400 3300 60  0000 C CNN
-F 3 "" H 7400 3300 60  0000 C CNN
-	1    7400 3300
-	1    0    0    -1
-$EndComp
 $Comp
 L CC3000 IC1
@@
 	1    0    0    -1
 $EndComp
+$Comp
+L TM4C1230H6PM U1
+U 1 1 5398E33D
+P 8100 3200
+F 0 "U1" H 6950 4950 45  0000 C CNN
+F 1 "TM4C1230H6PM" H 9050 1400 45  0000 C CNN
+F 2 "LQFP64" H 8100 3200 35  0000 C CIN
+F 3 "" H 8100 3900 60  0000 C CNN
+	1    8100 3200
+	1    0    0    -1
+$EndComp

Commit message: only 2 things wrong, missing button
Parts:
- removed U1: TM4C1230H6PM, LQFP64, symbol TM4C1230H6PM
- added A1: ANT, lifesense:ant_Wigle_A2_4G, symbol ANT
- added C10, C11, C18, C3, C5, C8: 0.01uF, lifesense:SMD-0603_c, symbol C
- added C100: 4.7uF, lifesense:SMD-0603_c, symbol C
- added C101: 1pF, lifesense:SMD-0603_c, symbol C
- added C102: 100nF, lifesense:SMD-0603_c, symbol C
- added C12, C14, C7: 1.0uF, lifesense:SMD-0603_c, symbol C
- added C22: 2.2uF, lifesense:SMD-0603_c, symbol C
- added C28, C29: 24pF, lifesense:SMD-0603_c, symbol C
- added C31, C32: 10pF, lifesense:SMD-0603_c, symbol C
- added C4, C6: 0.1uF, lifesense:SMD-0603_c, symbol C
- added CON1: USB-MINI-B, lifesense:ZX62-AB-5PA(11), symbol USB-MINI-B
- added D2, D3: LED, LEDs:LED-0805, symbol LED
- added D4: Green, LEDs:LED-0805, symbol LED
- added J1, J4: CONN_10X2, Pin_Headers:Pin_Header_Straight_2x10, symbol CONN_10X2
- added P1: CONN_6, Pin_Headers:Pin_Header_Straight_1x06, symbol CONN_6
- added P2, P21: CONN_01X01, lifesense:Pin_Header_Straight_1x01, symbol CONN_01X01
- added Q1, Q2, Q3: DTC114E, lifesense:DTC114EET1G, symbol DTC114E
- added R10, R11, R12, R14, R2, R25, R26, R29, R9: R, lifesense:SMD-0603_r, symbol R
- added R13: 0, lifesense:SMD-0603_r, symbol R
- added R27, R3, R4, R5, R8: 330, lifesense:SMD-0603_r, symbol R
- added R28: 10K, lifesense:SMD-0603_r, symbol R
- added R31: 1M, lifesense:SMD-0603_r, symbol R
- added SW1, SW2, SW3: SW_PUSH, symbol SW_PUSH
- added U1: TM4C123GH6PM, lifesense:lqfp64, symbol TM4C123GH6PM
- added U2: TPS73633DRB, lifesense:TPS73633DBV, symbol TPS73633DRB
- added Y1: CRYSTAL, lifesense:AB26TRB, symbol CRYSTAL
- added Y2: CRYSTAL, lifesense:ABM3, symbol CRYSTAL
- D1: footprint (none) -> LEDs:LED-0805
- IC1: footprint (none) -> texas-addition:CC3000
- R1: value R -> 0; footprint (none) -> lifesense:SMD-0603_r
Connections:
- net labels added: +3.3V, LED_B, LED_G, LED_R, MCU_PWR, MCU_VDDC, MISO, MOSI, PA0, PA1, PA2, PA3, PA4, PA5, PA6, PA7, PB0, PB1, PB2, PB3, PB4, PB5, PB6, PB7, PC0, PC1, PC2, PC3, PC4, PC5, PC6, PC7, PD0, PD1, PD2, PD3, PD6, PD7, PE0, PE1, PE2, PE3, PE4, PE5, PF0, PF1, PF2, PF3, PF4, SCK, SPI_CS, SPI_INT, USB_DM, USB_DP, USB_VBUS, USR_SW1, USR_SW2, VBAT_SW, ~HIB~, ~RST~, ~WAKE~
- net labels removed: VCC
- wire segments 3 -> 292
Other:
- moved on the sheet: IC1

Commit message: finished board 1.0
Parts:
- removed R1, R13: 0, lifesense:SMD-0603_r, symbol R
- removed R8: 330, lifesense:SMD-0603_r, symbol R
- removed SW1, SW2: SW_PUSH, symbol SW_PUSH
Connections:
- net labels removed: USR_SW1, USR_SW2
- wire segments 292 -> 278

Commit message: fabricated 1.1 version
Parts:
- removed U2: TPS73633DRB, lifesense:TPS73633DBV, symbol TPS73633DRB
- added U2: TPS73633DBV, symbol TPS73633DBV
Connections:
- wire segments 278 -> 280
Changed lines of the file:
@@
-$EndComp
-$Comp
-L TPS73633DRB U2
-U 1 1 53ED8F06
-P 10300 1150
-F 0 "U2" H 10050 1450 40  0000 C CNN
-F 1 "TPS73633DRB" H 10450 1450 40  0000 C CNN
-F 2 "lifesense:TPS73633DBV" H 9900 1600 30  0001 C CIN
-F 3 "" H 10300 1150 60  0000 C CNN
-	1    10300 1150
-	1    0    0    -1
 $EndComp
 $Comp
@@
 F 3 "" H 5250 2250 60  0000 C CNN
 	1    5250 2250
-	1    0    0    -1
+	-1   0    0    1
 $EndComp
 $Comp
@@
 F 3 "" H 5250 2900 60  0000 C CNN
 	1    5250 2900
-	1    0    0    -1
+	-1   0    0    1
 $EndComp
 $Comp
@@
 F 3 "" H 5250 3500 60  0000 C CNN
 	1    5250 3500
-	1    0    0    -1
-$EndComp
-$Comp
-L GND #PWR029
-U 1 1 53EE9E3D
-P 5600 2300
-F 0 "#PWR029" H 5600 2300 30  0001 C CNN
-F 1 "GND" H 5600 2230 30  0001 C CNN
-F 2 "" H 5600 2300 60  0000 C CNN
-F 3 "" H 5600 2300 60  0000 C CNN
-	1    5600 2300
-	1    0    0    -1
-$EndComp
-$Comp
-L GND #PWR030
-U 1 1 53EE9E51
-P 5600 2950
-F 0 "#PWR030" H 5600 2950 30  0001 C CNN
-F 1 "GND" H 5600 2880 30  0001 C CNN
-F 2 "" H 5600 2950 60  0000 C CNN
-F 3 "" H 5600 2950 60  0000 C CNN
-	1    5600 2950
-	1    0    0    -1
-$EndComp
-$Comp
-L GND #PWR031
-U 1 1 53EE9E65
-P 5600 3550
-F 0 "#PWR031" H 5600 3550 30  0001 C CNN
-F 1 "GND" H 5600 3480 30  0001 C CNN
-F 2 "" H 5600 3550 60  0000 C CNN
-F 3 "" H 5600 3550 60  0000 C CNN
-	1    5600 3550
-	1    0    0    -1
+	-1   0    0    1
 $EndComp
 $Comp
@@
 $EndComp
 $Comp
-L GND #PWR032
+L GND #PWR029
 U 1 1 53EEC6FF
 P 4050 4050
-F 0 "#PWR032" H 4050 4050 30  0001 C CNN
+F 0 "#PWR029" H 4050 4050 30  0001 C CNN
 F 1 "GND" H 4050 3980 30  0001 C CNN
 F 2 "" H 4050 4050 60  0000 C CNN
@@
 $EndComp
 $Comp
-L GND #PWR033
+L GND #PWR030
 U 1 1 53EEC743
 P 4050 3350
-F 0 "#PWR033" H 4050 3350 30  0001 C CNN
+F 0 "#PWR030" H 4050 3350 30  0001 C CNN
 F 1 "GND" H 4050 3280 30  0001 C CNN
 F 2 "" H 4050 3350 60  0000 C CNN
@@
 $EndComp
 $Comp
-L GND #PWR034
+L GND #PWR031
 U 1 1 53EEC780
 P 4050 2700
-F 0 "#PWR034" H 4050 2700 30  0001 C CNN
+F 0 "#PWR031" H 4050 2700 30  0001 C CNN
 F 1 "GND" H 4050 2630 30  0001 C CNN
 F 2 "" H 4050 2700 60  0000 C CNN
@@
 $EndComp
 $Comp
-L GND #PWR035
+L GND #PWR032
 U 1 1 53F3E3C0
 P 950 3900
-F 0 "#PWR035" H 950 3900 30  0001 C CNN
+F 0 "#PWR032" H 950 3900 30  0001 C CNN
 F 1 "GND" H 950 3830 30  0001 C CNN
 F 2 "" H 950 3900 60  0000 C CNN
@@
 $EndComp
 $Comp
-L GND #PWR036
+L GND #PWR033
 U 1 1 53F3EF4F
 P 3650 7550
-F 0 "#PWR036" H 3650 7550 30  0001 C CNN
+F 0 "#PWR033" H 3650 7550 30  0001 C CNN
 F 1 "GND" H 3650 7480 30  0001 C CNN
 F 2 "" H 3650 7550 60  0000 C CNN
@@
 $EndComp
 $Comp
-L +3.3V #PWR037
+L +3.3V #PWR034
 U 1 1 53F404D6
 P 3950 5850
-F 0 "#PWR037" H 3950 5810 30  0001 C CNN
+F 0 "#PWR034" H 3950 5810 30  0001 C CNN
 F 1 "+3.3V" H 3950 5960 30  0000 C CNN
 F 2 "" H 3950 5850 60  0000 C CNN
@@
 SCK
 $Comp
-L GND #PWR038
+L GND #PWR035
 U 1 1 53FE1F52
 P 9550 1800
-F 0 "#PWR038" H 9550 1800 30  0001 C CNN
+F 0 "#PWR035" H 9550 1800 30  0001 C CNN
 F 1 "GND" H 9550 1730 30  0001 C CNN
 F 2 "" H 9550 1800 60  0000 C CNN
@@
 $EndComp
 $Comp
-L GND #PWR039
+L GND #PWR036
 U 1 1 53FE39C3
 P 7950 6600
-F 0 "#PWR039" H 7950 6600 30  0001 C CNN
+F 0 "#PWR036" H 7950 6600 30  0001 C CNN
 F 1 "GND" H 7950 6530 30  0001 C CNN
 F 2 "" H 7950 6600 60  0000 C CNN
@@
 MISO
 $Comp
-L USB_VBUS #PWR040
+L USB_VBUS #PWR037
 U 1 1 53FF94E7
 P 2300 1300
-F 0 "#PWR040" H 2300 1400 30  0001 C CNN
+F 0 "#PWR037" H 2300 1400 30  0001 C CNN
 F 1 "USB_VBUS" H 2300 1410 30  0000 C CNN
 F 2 "" H 2300 1300 60  0000 C CNN
@@
 $EndComp
 $Comp
-L GND #PWR041
+L GND #PWR038
 U 1 1 53FFB6BD
 P 7650 6600
-F 0 "#PWR041" H 7650 6600 30  0001 C CNN
+F 0 "#PWR038" H 7650 6600 30  0001 C CNN
 F 1 "GND" H 7650 6530 30  0001 C CNN
 F 2 "" H 7650 6600 60  0000 C CNN
@@
 $EndComp
 $Comp
-L GND #PWR042
+L GND #PWR039
 U 1 1 53FFB703
 P 7750 6600
-F 0 "#PWR042" H 7750 6600 30  0001 C CNN
+F 0 "#PWR039" H 7750 6600 30  0001 C CNN
 F 1 "GND" H 7750 6530 30  0001 C CNN
 F 2 "" H 7750 6600 60  0000 C CNN
@@
 $EndComp
 $Comp
-L GND #PWR043
+L GND #PWR040
 U 1 1 53FFB749
 P 7850 6600
-F 0 "#PWR043" H 7850 6600 30  0001 C CNN
+F 0 "#PWR040" H 7850 6600 30  0001 C CNN
 F 1 "GND" H 7850 6530 30  0001 C CNN
 F 2 "" H 7850 6600 60  0000 C CNN
@@
 $EndComp
 $Comp
-L GND #PWR044
+L GND #PWR041
 U 1 1 53FFB78F
 P 8150 6600
-F 0 "#PWR044" H 8150 6600 30  0001 C CNN
+F 0 "#PWR041" H 8150 6600 30  0001 C CNN
 F 1 "GND" H 8150 6530 30  0001 C CNN
 F 2 "" H 8150 6600 60  0000 C CNN
@@
 $EndComp
 Wire Wire Line
-	5600 3500 5600 3550
-Wire Wire Line
-	5450 3500 5600 3500
+	5600 3500 5450 3500
 Wire Wire Line
 	4900 3500 5050 3500
-Wire Wire Line
-	5600 2900 5600 2950
-Wire Wire Line
-	5450 2900 5600 2900
-Wire Wire Line
-	5600 2250 5600 2300
 Wire Wire Line
 	5450 2250 5600 2250
@@
 Wire Wire Line
 	10750 1150 10850 1150
-Connection ~ 10200 1500
 Wire Wire Line
 	10200 1450 10200 1600
-Wire Wire Line
-	10350 1500 10200 1500
-Wire Wire Line
-	10350 1450 10350 1500
 Wire Wire Line
 	9850 1150 9650 1150
@@
 Wire Wire Line
 	3950 1200 4050 1200
+$Comp
+L TPS73633DBV U2
+U 1 1 54147A3C
+P 10300 1150
+F 0 "U2" H 10050 1450 40  0000 C CNN
+F 1 "TPS73633DBV" H 10450 1450 40  0000 C CNN
+F 2 "" H 9900 1600 30  0000 C CIN
+F 3 "" H 10300 1150 60  0000 C CNN
+	1    10300 1150
+	1    0    0    -1
+$EndComp
+Wire Wire Line
+	3500 4750 3650 4750
+Wire Wire Line
+	3650 4750 3650 4850
+Wire Wire Line
+	3650 4850 3500 4850
+Wire Wire Line
+	3500 5050 3650 5050
+Wire Wire Line
+	3650 5050 3650 5150
+Wire Wire Line
+	3650 5150 3500 5150
+$Comp
+L USB_VBUS #PWR042
+U 1 1 5414C346
+P 5600 2050
+F 0 "#PWR042" H 5600 2150 30  0001 C CNN
+F 1 "USB_VBUS" H 5600 2160 30  0000 C CNN
+F 2 "" H 5600 2050 60  0000 C CNN
+F 3 "" H 5600 2050 60  0000 C CNN
+	1    5600 2050
+	1    0    0    -1
+$EndComp
+Wire Wire Line
+	5600 2050 5600 3500
+Wire Wire Line
+	5450 2900 5600 2900
+Connection ~ 5600 2900
+Connection ~ 5600 2250
 $EndSCHEMATC
